File: libreboard.kicad_sch (KiCad schematic)
At the start: 66 parts, among them J100 Screw Terminal, J101 Screw Terminal, J11 USB_C_Receptacle_USB2.0, J51 12V Fan 1, J52 12V Fan 2, J53 12V Fan 3, J54 12V Fan 4, U10 EMC2305-x-AP, U14 PTPS55289RYQR, U4 PTPS55289RYQR

Commit message: cleanup, testpoints
Parts:
- added TP2: TestPoint 12V, TestPoint:TestPoint_Pad_D1.5mm, symbol Connector:TestPoint
- added TP4, TP7: TestPoint GND, TestPoint:TestPoint_Pad_D1.5mm, symbol Connector:TestPoint
- added TP6: TestPoint +5V, TestPoint:TestPoint_Pad_D1.5mm, symbol Connector:TestPoint
- J54: now fitted
Connections:
- net +12V: now also TP2.1
- net +5v: now also TP6.1
- net GND: now also TP4.1, TP7.1

Commit message: cleanup, testpoints
Connections:
- net GND: no longer U4.2 (MODE)
- net at C23.1, U4.18 (VCC), U4.21 (EXTVCC): now also U4.2 (MODE)
Other:
- moved on the sheet: C20, C21, C22, C23, C24, C25, C26, C27, C28, C29, C30, C51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
