File: libreboard.kicad_sch (KiCad schematic)
At the start: 77 parts, among them J100 Screw Terminal, J101 Screw Terminal, J11 USB_C_Receptacle_USB2.0, J51 12V Fan 1, J52 12V Fan 2, J53 12V Fan 3, J54 12V Fan 4, U10 EMC2305-x-AP, U14 TPS552892RYQR, U4 TPS552892RYQR

Commit message: Power: C66-C68 are real 47 uF caps on U14's +5v output
C66-C68 (U14 output, CM5 +5v) were drawn as 47 uF in 0603 in
7a278c5. The BOM pass in e28bff3 gave them Wurth 885012005011, a
47 pF C0G 0402 part, and shrank the footprint to 0402; the value field
kept saying 47 uF. The same pass also put U4's 33 uF outputs (C27-C29)
in 0402 (fixed to TDK 1206 in 9f53362) and 6.3 V parts on the 12-24 V
input (C21/C52, fixed in Rev2) and on +12V (C30, fixed in a2bb35c);
C66-C68 were missed, so Rev1 has about 47 pF of ceramic output
capacitance where ~140 uF was intended, leaving the 270 uF polymer
C69 alone.

Now TDK C3216X5R1A476M160AB, 47 uF 10 V X5R 1206, mirroring U4's
C27-C29. Digikey number left blank (not verified). Connectivity
unchanged; ERC unchanged at 346.

Co-Authored-By: Claude Opus 5.5 <noreply@anthropic.com>
Parts:
- C66, C67, C68: footprint Capacitor_SMD:C_0402_1005Metric -> Capacitor_SMD:C_1206_3216Metric; Dist. P/N 732-7429-2-ND -> (none); Manf. P/N 885012005011 -> C3216X5R1A476M160AB; Manufacturer Würth Elektronik -> TDK Corporation; Part Description Capacitor, Ceramic, 47pF, ±5%, 10V, C0G/NP0, 0402 (1005m) -> 47 µF ±20% 10V Ceramic Capacitor X5R 1206 (3216 Metric)
Changed lines of the file:
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@@
 			)
 		)
-		(property "Footprint" "Capacitor_SMD:C_0402_1005Metric"
+		(property "Footprint" "Capacitor_SMD:C_1206_3216Metric"
 			(at 270.51 344.17 0)
 			(hide yes)
@@
 			)
 		)
-		(property "Dist. P/N" "732-7429-2-ND"
+		(property "Dist. P/N" ""
 			(at 270.51 344.17 0)
 			(hide yes)
@@
 			)
 		)
-		(property "Manf. P/N" "885012005011"
+		(property "Manf. P/N" "C3216X5R1A476M160AB"
 			(at 270.51 344.17 0)
 			(hide yes)
@@
 			)
 		)
-		(property "Manufacturer" "Würth Elektronik"
+		(property "Manufacturer" "TDK Corporation"
 			(at 270.51 344.17 0)
 			(hide yes)
@@
 			)
 		)
-		(property "Part Description" "Capacitor, Ceramic, 47pF, ±5%, 10V, C0G/NP0, 0402 (1005m)"
+		(property "Part Description" "47 µF ±20% 10V Ceramic Capacitor X5R 1206 (3216 Metric)"
 			(at 270.51 344.17 0)
 			(hide yes)
@@
 			)
 		)
-		(property "Footprint" "Capacitor_SMD:C_0402_1005Metric"
+		(property "Footprint" "Capacitor_SMD:C_1206_3216Metric"
 			(at 281.94 344.17 0)
 			(hide yes)
@@
 			)
 		)
-		(property "Dist. P/N" "732-7429-2-ND"
+		(property "Dist. P/N" ""
 			(at 281.94 344.17 0)
 			(hide yes)
@@
 			)
 		)
-		(property "Manf. P/N" "885012005011"
+		(property "Manf. P/N" "C3216X5R1A476M160AB"
 			(at 281.94 344.17 0)
 			(hide yes)
@@
 			)
 		)
-		(property "Manufacturer" "Würth Elektronik"
+		(property "Manufacturer" "TDK Corporation"
 			(at 281.94 344.17 0)
 			(hide yes)
@@
 			)
 		)
-		(property "Part Description" "Capacitor, Ceramic, 47pF, ±5%, 10V, C0G/NP0, 0402 (1005m)"
+		(property "Part Description" "47 µF ±20% 10V Ceramic Capacitor X5R 1206 (3216 Metric)"
 			(at 281.94 344.17 0)
 			(hide yes)
@@
 			)
 		)
-		(property "Footprint" "Capacitor_SMD:C_0402_1005Metric"
+		(property "Footprint" "Capacitor_SMD:C_1206_3216Metric"
 			(at 292.1 344.17 0)
 			(hide yes)
@@
 			)
 		)
-		(property "Dist. P/N" "732-7429-2-ND"
+		(property "Dist. P/N" ""
 			(at 292.1 344.17 0)
 			(hide yes)
@@
 			)
 		)
-		(property "Manf. P/N" "885012005011"
+		(property "Manf. P/N" "C3216X5R1A476M160AB"
 			(at 292.1 344.17 0)
 			(hide yes)
@@
 			)
 		)
-		(property "Manufacturer" "Würth Elektronik"
+		(property "Manufacturer" "TDK Corporation"
 			(at 292.1 344.17 0)
 			(hide yes)
@@
 			)
 		)
-		(property "Part Description" "Capacitor, Ceramic, 47pF, ±5%, 10V, C0G/NP0, 0402 (1005m)"
+		(property "Part Description" "47 µF ±20% 10V Ceramic Capacitor X5R 1206 (3216 Metric)"
 			(at 292.1 344.17 0)
 			(hide yes)

Commit message: HUB_3V3 also feeds the status LEDs, R52 and the TCA9538
The hub-side 3.3 V copper on the PCB also runs on to D1/D2/U5, R52
and U17/R4, so those move onto the hub's always-on rail too:

- U5 + D1 (red power LED): the CM5's LED_nPWR is meant to light the
  red LED while the board is powered but shut down, and the CM5's
  3.3 V output is off exactly then (CM5 datasheet, pins 84/86), so the
  standby LED never worked. On HUB_3V3 it can.
- D2 (green ACT LED): LED_nACT is 5 V tolerant open drain, so no
  back-powering into a shut-down CM5.
- R52 (U16 OE# pull-up): U16 runs from +5v; on HUB_3V3 the LED gate
  stays shut while the CM5's 3.3 V is still down at boot.
- U17 TCA9538 + R4: same rail as the hub reset (U19 MR) and LED gate
  it drives; I2C pins are open drain, no back-powering. The expander
  now keeps its register state across CM5 shutdowns (resets on +5v).

HUB_3V3 becomes a top-level net (/HUB_3V3): hierarchical labels on
the CM5_HighSpeed (U20 output) and CM5_GPIO sheets, sheet pins and a
labelled wire on the root sheet. 15 nodes on /HUB_3V3; /+3.3v keeps
the camera, J15 Rp, fan controller, I2C pull-ups, SD switch, header,
Qwiic and Ethernet LEDs. ERC unchanged at 346.

Co-Authored-By: Claude Opus 5.5 <noreply@anthropic.com>
Other:
- sheet CM5_GPIO ( Ethernet, GPIO, SDCARD) ports: added HUB_3V3; removed none
- sheet CM5_HighSpeed ports: added HUB_3V3; removed none
Changed lines of the file:
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@@
 	(wire
 		(pts
+			(xy 165.1 96.52) (xy 165.1 111.76)
+		)
+		(stroke
+			(width 0)
+			(type default)
+		)
+	)
+	(wire
+		(pts
 			(xy 320.04 342.9) (xy 327.66 342.9)
 		)
@@
 		)
 	)
+	(label "HUB_3V3"
+		(at 165.1 106.68 90)
+		(effects
+			(font
+				(size 1.27 1.27)
+			)
+			(justify left bottom)
+		)
+	)
 	(symbol
 		(lib_id "Mechanical:MountingHole")
@@
 			)
 		)
+		(pin "HUB_3V3" input
+			(at 165.1 111.76 90)
+			(effects
+				(font
+					(size 1.27 1.27)
+				)
+				(justify right)
+			)
+		)
 		(instances
 			(project "libreboard"
@@
 					(size 1.27 1.27)
 				)
-				(justify left)
+				(justify right)
 			)
 		)
@@
 			(effects
 				(font
+					(size 1.27 1.27)
+				)
+				(justify left)
+			)
+		)
+		(pin "HUB_3V3" output
+			(at 165.1 96.52 270)
+			(effects
+				(font

Commit message: BOM: LCSC codes for JLCPCB assembly, DigiKey numbers verified
Sourcing pass for a rev3 build at JLCPCB (SMT + through-hole), keeping
the DigiKey BOM usable. Report and per-part data in bom/rev3-sourcing.*.

- New hidden "LCSC" field on 189 parts (88 of 93 part numbers).
  Passives use JLC Basic/Preferred equivalents where value, size,
  tolerance, voltage and dielectric match or improve (0402 resistors at
  62.5 mW: worst-case dissipation on this board < 5 mW); ICs and
  connectors use the exact part. Exact codes are stored even where JLC
  has no stock (U4/U14, U3, U16, U17, BT1) - see the report.
- DigiKey: every existing number checked against its MPN (reel numbers
  kept). Filled: J7 (was Farnell 2358234), C60 (AVX new PN
  KGM05ACG1H6R8CH), C61, C66-C68, Q1/Q2, U20, U21. C73: wrong number
  (490-1494-2-ND is GRM188R71H102KA01D) cleared - to fill by hand.
- C72: Murata GRM188R71C104KA01D is obsolete -> Yageo CC0603KRX7R9BB104
  (0.1 uF 50 V X7R 0603).
- Fixes: L2/L3 manufacturer Coilcraft -> Bourns; U9 distributor typo
  LSCS -> LCSC; C27-C29 DigiKey number without " - Cut Tape" suffix.

Not yet stored: Y1, J2, J8, SW1/SW2 candidates need review; M1 is a
screw. Connectivity, values and footprints unchanged; ERC unchanged
at 342.

Co-Authored-By: Claude Opus 5.5 <noreply@anthropic.com>
Parts:
- C18, C31, C9: LCSC (none) -> C1525
- C20: LCSC (none) -> C7059708
- C21, C52: LCSC (none) -> C440198
- C22, C30, C54: LCSC (none) -> C1518208
- C23, C53: LCSC (none) -> C29823
- C24, C25, C55, C65: LCSC (none) -> C307331
- C26: LCSC (none) -> C2162042
- C27, C28, C29: Dist. P/N 445-8046-1-ND - Cut Tape -> 445-8046-1-ND; LCSC (none) -> C342307
- C51: LCSC (none) -> C46550474
- C60: Dist. P/N (none) -> 478-KGM05ACG1H6R8CHTR-ND; LCSC (none) -> C1576
- C61: Dist. P/N (none) -> 490-3244-2-ND; LCSC (none) -> C76947
- C62: LCSC (none) -> C1531
- C63: LCSC (none) -> C1517504
- C64: LCSC (none) -> C52923
- C66, C67, C68: Dist. P/N (none) -> 445-6006-2-ND; LCSC (none) -> C96123
- C69: LCSC (none) -> C2944013
- J100, J101: LCSC (none) -> C5187194
- J11: LCSC (none) -> C3020560
- J51, J52, J53, J54: LCSC (none) -> C240840
- L2, L3: LCSC (none) -> C6685196; Manufacturer Coilcraft -> Bourns
- R11: LCSC (none) -> C2986234
- R13: LCSC (none) -> C7501196
- R18, R6: LCSC (none) -> C7209900
- R19, R7: LCSC (none) -> C2986582
- R20: LCSC (none) -> C2076811
- R21, R22, R23, R24, R29, R30: LCSC (none) -> C25744
- R31: LCSC (none) -> C25768
- R32: LCSC (none) -> C25779
- R53, R55: LCSC (none) -> C25741
- R54: LCSC (none) -> C2076806
- R56: LCSC (none) -> C409880
- R8: LCSC (none) -> C2077134
- U10: LCSC (none) -> C621415
- U14, U4: LCSC (none) -> C19272254

Commit message: BOM: JLC sourcing decisions (U4/U14, U16, U17, BT1, Y1, J2, J8, SW1/SW2)
Michael's decisions on bom/rev3-sourcing.md section 1:
- U4/U14: TPS552892RYQR (unobtainable) -> TPS552892QWRYQRQ1, the
  AEC-Q100 version (same pins, RYQ package, VREF, input range).
  To be bought at Mouser and supplied to JLC (JLC and DigiKey 0).
- U16: SOT-553 DRLR (0 at JLC) -> SC-70-5 SN74AHCT1G125DCKR
  (C350557), same pinout; SC-70-5 because U16 is 1.5-2.3 mm from
  C71/C70/R9/R52. Footprint Package_TO_SOT_SMD:SOT-353_SC-70-5.
- U17 TCA9538DBR: hand-fitted from DigiKey; in_pos_files no /
  exclude_from_pos_files.
- BT1: Linx BAT-HLD-007-SMT-TR -> Keystone 3000TR (C6997853), the
  12 mm retainer it copies: + tabs at +-7.9 mm, - is the board pad,
  so the footprint stays.
- Y1: ECS-2520MV-240-DN-TR -> YXC OT252024MJBA4SL (C669072). YXC
  datasheet: pin 1 tri-state enabled when floating (Y1 pin 1 is NC),
  pins 2/3/4 GND/OUT/VDD as on the ECS part, 1.8-3.3 V, same 2520
  land pattern.
- J2: Molex 0010897140 -> 0010897142 (C561778), same header and pin
  lengths with 15 uin instead of 30 uin gold (Mouser 538-10-89-7142).
- J8: Molex 0010897400 -> Wurth 61304021121 (C5364405, 732-5310-ND);
  insulator 0.25 mm taller.
- SW1/SW2: C&K PTS645VH58-2 LFS -> PTS645VK39-2 LFS (C285519,
  CKN10053-ND); footprints -> PTS645Vx39-2LFS (same pads as the
  Vx58/Vx31 ones used before).
- TUSB4041 kept; M2-M5 nuts fitted by hand.

Fields mirrored on the PCB footprints where the footprint does not
change. U16 and SW1/SW2 need F8 (Replace footprints); U16 then needs
re-routing. ERC unchanged at 342; DRC parity differs only by those
three footprint swaps.

Co-Authored-By: Claude Opus 5.5 <noreply@anthropic.com>
Parts:
- U14, U4: value TPS552892RYQR -> TPS552892QWRYQRQ1; Dist. P/N 296-TPS552892RYQRTR-ND -> 296-TPS552892QWRYQRQ1TR-ND; LCSC C19272254 -> C22375748; Manf. P/N TPS552892RYQR -> TPS552892QWRYQRQ1
Changed lines of the file:
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@@
 			)
 		)
-		(property "Value" "TPS552892RYQR"
+		(property "Value" "TPS552892QWRYQRQ1"
 			(at 195.58 186.69 0)
 			(show_name no)
@@
 			)
 		)
-		(property "Datasheet" "https://www.ti.com/lit/ds/symlink/tps552892.pdf"
+		(property "Datasheet" "https://www.ti.com/lit/ds/symlink/tps552892-q1.pdf"
 			(at 173.99 194.31 0)
 			(hide yes)
@@
 			)
 		)
-		(property "Dist. P/N" "296-TPS552892RYQRTR-ND"
+		(property "Dist. P/N" "296-TPS552892QWRYQRQ1TR-ND"
 			(at 173.99 194.31 0)
 			(hide yes)
@@
 			)
 		)
-		(property "Manf. P/N" "TPS552892RYQR"
+		(property "Manf. P/N" "TPS552892QWRYQRQ1"
 			(at 173.99 194.31 0)
 			(hide yes)
@@
 			)
 		)
-		(property "LCSC" "C19272254"
+		(property "LCSC" "C22375748"
 			(at 173.99 194.31 0)
 			(hide yes)
@@
 			)
 		)
-		(property "Value" "TPS552892RYQR"
+		(property "Value" "TPS552892QWRYQRQ1"
 			(at 199.39 298.45 0)
 			(show_name no)
@@
 			)
 		)
-		(property "Datasheet" "https://www.ti.com/lit/ds/symlink/tps552892.pdf"
+		(property "Datasheet" "https://www.ti.com/lit/ds/symlink/tps552892-q1.pdf"
 			(at 177.8 306.07 0)
 			(hide yes)
@@
 			)
 		)
-		(property "Dist. P/N" "296-TPS552892RYQRTR-ND"
+		(property "Dist. P/N" "296-TPS552892QWRYQRQ1TR-ND"
 			(at 177.8 306.07 0)
 			(hide yes)
@@
 			)
 		)
-		(property "Manf. P/N" "TPS552892RYQR"
+		(property "Manf. P/N" "TPS552892QWRYQRQ1"
 			(at 177.8 306.07 0)
 			(hide yes)
@@
 			)
 		)
-		(property "LCSC" "C19272254"
+		(property "LCSC" "C22375748"
 			(at 177.8 306.07 0)
 			(hide yes)

Commit message: Fan controller: 10k pull-up on unused TACH5; ERC drawing cleanup
From the ERC review (342 messages, none an electrical fault):
- U10 (EMC2305) TACH5, pin 16, was floating. The datasheet types the
  TACH inputs as open-drain inputs that need an external pull-up, so
  it gets the same 10k to +3.3v as TACH1-4: new R64 (ERJ-U02F1002X,
  LCSC C25744) above R21-R24 on the +3.3v bus, joined to pin 16 by a
  TACH5 label. No-connect flags on the unused PWM5 (pin 15) and
  ALERT# (pin 12) outputs.
- Removed the two GPIO_VREF sheet pins on the root sheet and the wire
  between them: neither sub-sheet has that label and the wire joined
  only those two pins. The CM5's GPIO_VREF pin is on +3.3v inside
  CM5_GPIO as before.
- Removed a no-connect flag in CM5_GPIO at (185.42, 118.11) that has
  never been on a pin.

Netlist: only R64 (+3.3v / TACH5) and U10 pin 16 (-> TACH5) change.
ERC 340 -> 333. PCB needs F8 to add R64 (0402) near U10, plus routing.

Co-Authored-By: Claude Opus 5.5 <noreply@anthropic.com>
Parts:
- added R64: 10kΩ, Resistor_SMD:R_0402_1005Metric, symbol Device:R_Small
Connections:
- net +3.3v: now also R64.1
- net TACH5: now reaches U10.16 (TACH5)
- net TACH5: now also R64.2
- no-connect marks 9 -> 11
Other:
- sheet CM5_GPIO ( Ethernet, GPIO, SDCARD) ports: added none; removed GPIO_VREF
- sheet CM5_HighSpeed ports: added none; removed GPIO_VREF
Changed lines of the file:
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@@
 	(wire
 		(pts
-			(xy 180.34 96.52) (xy 180.34 111.76)
-		)
-		(stroke
-			(width 0)
-			(type solid)
-		)
-	)
-	(wire
-		(pts
 			(xy 71.12 121.92) (xy 74.93 121.92)
 		)
@@
 		)
 	)
+	(wire
+		(pts
+			(xy 58.42 111.76) (xy 58.42 113.03)
+		)
+		(stroke
+			(width 0)
+			(type default)
+		)
+	)
+	(wire
+		(pts
+			(xy 58.42 111.76) (xy 66.04 111.76)
+		)
+		(stroke
+			(width 0)
+			(type default)
+		)
+	)
+	(wire
+		(pts
+			(xy 71.12 111.76) (xy 73.66 111.76)
+		)
+		(stroke
+			(width 0)
+			(type default)
+		)
+	)
+	(wire
+		(pts
+			(xy 71.12 162.56) (xy 73.66 162.56)
+		)
+		(stroke
+			(width 0)
+			(type default)
+		)
+	)
+	(junction
+		(at 58.42 113.03)
+		(diameter 0)
+		(color 0 0 0 0)
+	)
+	(label "TACH5"
+		(at 73.66 111.76 0)
+		(effects
+			(font
+				(size 1.27 1.27)
+			)
+			(justify left bottom)
+		)
+	)
+	(label "TACH5"
+		(at 73.66 162.56 0)
+		(effects
+			(font
+				(size 1.27 1.27)
+			)
+			(justify left bottom)
+		)
+	)
+	(no_connect
+		(at 71.12 160.02)
+	)
+	(no_connect
+		(at 45.72 157.48)
+	)
+	(symbol
+		(lib_id "Device:R_Small")
+		(at 68.58 111.76 90)
+		(unit 1)
+		(body_style 1)
+		(exclude_from_sim no)
+		(in_bom yes)
+		(on_board yes)
+		(in_pos_files yes)
+		(dnp no)
+		(property "Reference" "R64"
+			(at 65.024 110.744 90)
+			(show_name no)
+			(do_not_autoplace no)
+			(effects
+				(font
+					(size 1.016 1.016)
+				)
+			)
+		)
+		(property "Value" "10kΩ"
+			(at 68.58 112.014 90)
+			(show_name no)
+			(do_not_autoplace no)
+			(effects
+				(font
+					(size 1.27 1.27)
+				)
+			)
+		)
+		(property "Footprint" "Resistor_SMD:R_0402_1005Metric"
+			(at 68.58 111.76 0)
+			(hide yes)
+			(show_name no)
+			(do_not_autoplace no)
+			(effects
+				(font
+					(size 1.27 1.27)
+				)
+			)
+		)
+		(property "Datasheet" ""
+			(at 68.58 111.76 0)
+			(hide yes)
+			(show_name no)
+			(do_not_autoplace no)
+			(effects
+				(font
+					(size 1.27 1.27)
+				)
+			)
+		)
+		(property "Description" "Resistor, small symbol"
+			(at 68.58 111.76 0)
+			(hide yes)
+			(show_name no)
+			(do_not_autoplace no)
+			(effects
+				(font
+					(size 1.27 1.27)
+				)
+			)
+		)
+		(property "Dist. P/N" "10-ERJ-U02F1002XTR-ND"
+			(at 68.58 111.76 90)
+			(hide yes)
+			(show_name no)
+			(do_not_autoplace no)
+			(effects
+				(font
+					(size 1.27 1.27)
+				)
+			)
+		)
+		(property "Distributor" "Digikey"
+			(at 68.58 111.76 90)
+			(hide yes)
+			(show_name no)
+			(do_not_autoplace no)
+			(effects
+				(font
+					(size 1.27 1.27)
+				)
+			)
+		)
+		(property "Manf. P/N" "ERJ-U02F1002X"
+			(at 68.58 111.76 90)
+			(hide yes)
+			(show_name no)
+			(do_not_autoplace no)
+			(effects
+				(font
+					(size 1.27 1.27)
+				)
+			)
+		)
+		(property "Manufacturer" "Panasonic"
+			(at 68.58 111.76 90)
+			(hide yes)
+			(show_name no)
+			(do_not_autoplace no)
+			(effects
+				(font
+					(size 1.27 1.27)
+				)
+			)
+		)
+		(property "Part Description" "Resistor, 10kΩ, ±1%, 0.1W, SMD 0402 (1005m)"
+			(at 68.58 111.76 90)
+			(hide yes)
+			(show_name no)
+			(do_not_autoplace no)
+			(effects
+				(font
+					(size 1.27 1.27)
+				)
+			)
+		)
+		(property "MANUFACTURER" ""
+			(at 68.58 111.76 90)
+			(hide yes)
+			(show_name no)
+			(do_not_autoplace no)
+			(effects
+				(font
+					(size 1.27 1.27)
+				)
+			)
+		)
+		(property "MAXIMUM_PACKAGE_HEIGHT" ""
+			(at 68.58 111.76 90)
+			(hide yes)
+			(show_name no)
+			(do_not_autoplace no)
+			(effects
+				(font
+					(size 1.27 1.27)
+				)
+			)
+		)
+		(property "PARTREV" ""
+			(at 68.58 111.76 90)
+			(hide yes)
+			(show_name no)
+			(do_not_autoplace no)
+			(effects
+				(font
+					(size 1.27 1.27)
+				)
+			)
+		)
+		(property "STANDARD" ""
+			(at 68.58 111.76 90)
+			(hide yes)
+			(show_name no)
+			(do_not_autoplace no)
+			(effects
+				(font
+					(size 1.27 1.27)
+				)
+			)
+		)
+		(property "LCSC" "C25744"
+			(at 68.58 111.76 0)
+			(hide yes)
+			(show_name no)
+			(do_not_autoplace no)
+			(effects
+				(font
+					(size 1.27 1.27)
+				)
+			)
+		)
+		(pin "1"
+		)
+		(pin "2"
+		)
+		(instances
+			(project "libreboard"
+				(path "/e63e39d7-6ac0-4ffd-8aa3-1841a4541b55"
+					(reference "R64")
+					(unit 1)
+				)
+			)
+		)
+	)
 	(symbol
 		(lib_id "Device:C_Small")
@@
 			)
 		)
-		(pin "GPIO_VREF" output
-			(at 180.34 111.76 90)
-			(effects
-				(font
-					(size 1.27 1.27)
-				)
-				(justify right)
-			)
-		)
 		(pin "CAM_GPIO0" output
 			(at 157.48 111.76 90)
@@
 			(effects
 				(font
-					(size 1.27 1.27)
-				)
-				(justify left)
-			)
-		)
-		(pin "GPIO_VREF" input
-			(at 180.34 96.52 270)
-			(effects
-				(font

Commit message: Freeze J11/J15/J7 symbols and J15 footprint in the project libraries
KiCad 10's stock library renamed the shield pin of
Connector:USB_C_Receptacle_USB2.0_16P (J11), USB_C_Receptacle (J15)
and Micro_SD_Card_Det2 (J7) from S1 / 11 to SH, and the stock
Connector_USB:USB_C_Receptacle_Molex_105450-0101 footprint now has SH
pads (and rounded pads). Our footprints use S1 / 11. Running "Update
symbols/footprints from library" would have left the shield pads of
these three connectors without their GND net.

- The three symbols, exactly as cached in the schematic, are now in
  libreboard.kicad_sym and the instances link there
  (libreboard:USB_C_Receptacle_USB2.0_16P, libreboard:USB_C_Receptacle,
  libreboard:Micro_SD_Card_Det2).
- J15's footprint, as placed on the board (28 pads, shields S1), is
  saved as libreboard:USB_C_Receptacle_Molex_105450-0101 and J15 links
  there in the schematic and on the board. J11 and J7 already used
  project footprints.

Netlist identical; ERC 333 -> 330 (the three lib_symbol_mismatch
warnings are gone); DRC with schematic parity unchanged.

Co-Authored-By: Claude Opus 5.5 <noreply@anthropic.com>
Parts:
- J11: symbol Connector:USB_C_Receptacle_USB2.0_16P -> libreboard:USB_C_Receptacle_USB2.0_16P
Changed lines of the file:
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@@
 	)
 	(symbol
-		(lib_id "Connector:USB_C_Receptacle_USB2.0_16P")
+		(lib_id "libreboard:USB_C_Receptacle_USB2.0_16P")
 		(at 46.99 59.69 0)
 		(unit 1)

Commit message: BOM: J11 to GCT USB4105-GF-A-120
JLC's stock of USB4105-GF-A (C3020560) dropped from 39 to 0. The -120
(C5184243, 1,153 at JLC; DigiKey 2073-USB4105-GF-A-120TR-ND) is the
same connector with 1.20 mm instead of 0.95 mm shell stakes; GCT's
drawing has one PCB layout for all stake lengths, and on the 1.6 mm
board the stakes do not come out the bottom. JLC's footprint matches
ours pad for pad. Fields only: ERC, DRC and schematic parity unchanged.

Co-Authored-By: Claude Opus 5.5 <noreply@anthropic.com>
Parts:
- J11: Dist. P/N 2073-USB4105-GF-ATR-ND -> 2073-USB4105-GF-A-120TR-ND; LCSC C3020560 -> C5184243; Manf. P/N USB4105-GF-A -> USB4105-GF-A-120
Changed lines of the file:
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@@
 			)
 		)
-		(property "Dist. P/N" "2073-USB4105-GF-ATR-ND"
+		(property "Dist. P/N" "2073-USB4105-GF-A-120TR-ND"
 			(at 46.99 59.69 0)
 			(hide yes)
@@
 			)
 		)
-		(property "Manf. P/N" "USB4105-GF-A"
+		(property "Manf. P/N" "USB4105-GF-A-120"
 			(at 46.99 59.69 0)
 			(hide yes)
@@
 			)
 		)
-		(property "LCSC" "C3020560"
+		(property "LCSC" "C5184243"
 			(at 46.99 59.69 0)
 			(hide yes)
