File: CM5_HighSpeed.kicad_sch (KiCad schematic)
At the start: 79 parts, among them J1 USB-C, J10 USB-C, J15 USB_C_Receptacle, J17 USB-C, J22 Conn_HDMI, J5 Conn_1x22_Female, J6 USB-C, Q1 2N7002, Q2 2N7002, U11 TUSB4041I, U12 RT9742SNGV, U13 TLV75712PDBVR, U15 AP22653W6, U19 TPS3808G01DBVR, U20 LP38693MP-3.3, U21 HD3SS3220RNHR, U6 AP22653W6, Y1 ECS-2520MV-240-CN-TR

Commit message: J15: C57 100 uF polymer (7343) -> 47 uF ceramic (1206)
With the HD3SS3220 gating, J15's VBUS only turns on after a device is
attached, so the USB 2.0 host-port 120 uF hot-plug reservoir is no
longer needed; a Type-C source needs >= 10 uF on VBUS. C57 becomes the
same 47 uF 10 V X5R 1206 as C66-C68 (TDK C3216X5R1A476M160AB,
445-6006-2-ND, LCSC C96123 Basic), freeing board space next to J15.
With C58/C59 (2 x 10 uF) the port keeps ~30-35 uF effective at 5 V.
Smaller VBUS capacitance also lets U15 discharge VBUS to vSafe0V faster,
so U21 can re-enable the port sooner after a re-plug.

Symbol Device:C_Polarized -> Device:C (same pin positions).
Connectivity unchanged; ERC unchanged at 342.

Co-Authored-By: Claude Opus 5.5 <noreply@anthropic.com>
Parts:
- C57: value 100µF -> 47µF; footprint Capacitor_Tantalum_SMD:CP_EIA-7343-31_Kemet-D -> Capacitor_SMD:C_1206_3216Metric; symbol Device:C_Polarized -> Device:C; Dist. P/N 399-11382-2-ND -> 445-6006-2-ND; LCSC C3275146 -> C96123; Manf. P/N A700X107M010ATE010 -> C3216X5R1A476M160AB; Manufacturer Kemet -> TDK Corporation; Part Description Capacitor, Aluminum, 100µF, ±20%, 10V, 10mΩ ESR -> 47 µF ±20% 10V Ceramic Capacitor X5R 1206 (3216 Metric)
Changed lines of the file:
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@@
 	)
 	(symbol
-		(lib_id "Device:C_Polarized")
+		(lib_id "Device:C")
 		(at 137.16 213.36 0)
 		(unit 1)
@@
 			)
 		)
-		(property "Value" "100µF"
+		(property "Value" "47µF"
 			(at 140.1572 214.503 0)
 			(show_name no)
@@
 			)
 		)
-		(property "Footprint" "Capacitor_Tantalum_SMD:CP_EIA-7343-31_Kemet-D"
+		(property "Footprint" "Capacitor_SMD:C_1206_3216Metric"
 			(at 138.1252 217.17 0)
 			(hide yes)
@@
 			)
 		)
-		(property "Description" "Polarized capacitor"
+		(property "Description" "Unpolarized capacitor"
 			(at 137.16 213.36 0)
 			(hide yes)
@@
 			)
 		)
-		(property "Part Description" "Capacitor, Aluminum, 100µF, ±20%, 10V, 10mΩ ESR"
+		(property "Part Description" "47 µF ±20% 10V Ceramic Capacitor X5R 1206 (3216 Metric)"
 			(at 137.16 213.36 0)
 			(hide yes)
@@
 			)
 		)
-		(property "Dist. P/N" "399-11382-2-ND"
+		(property "Dist. P/N" "445-6006-2-ND"
 			(at 137.16 213.36 0)
 			(hide yes)
@@
 			)
 		)
-		(property "Manf. P/N" "A700X107M010ATE010"
+		(property "Manf. P/N" "C3216X5R1A476M160AB"
 			(at 137.16 213.36 0)
 			(hide yes)
@@
 			)
 		)
-		(property "Manufacturer" "Kemet"
+		(property "Manufacturer" "TDK Corporation"
 			(at 137.16 213.36 0)
 			(hide yes)
@@
 			)
 		)
-		(property "LCSC" "C3275146"
+		(property "LCSC" "C96123"
 			(at 137.16 213.36 0)
 			(hide yes)

Commit message: BOM: JLC sourcing decisions (U4/U14, U16, U17, BT1, Y1, J2, J8, SW1/SW2)
Michael's decisions on bom/rev3-sourcing.md section 1:
- U4/U14: TPS552892RYQR (unobtainable) -> TPS552892QWRYQRQ1, the
  AEC-Q100 version (same pins, RYQ package, VREF, input range).
  To be bought at Mouser and supplied to JLC (JLC and DigiKey 0).
- U16: SOT-553 DRLR (0 at JLC) -> SC-70-5 SN74AHCT1G125DCKR
  (C350557), same pinout; SC-70-5 because U16 is 1.5-2.3 mm from
  C71/C70/R9/R52. Footprint Package_TO_SOT_SMD:SOT-353_SC-70-5.
- U17 TCA9538DBR: hand-fitted from DigiKey; in_pos_files no /
  exclude_from_pos_files.
- BT1: Linx BAT-HLD-007-SMT-TR -> Keystone 3000TR (C6997853), the
  12 mm retainer it copies: + tabs at +-7.9 mm, - is the board pad,
  so the footprint stays.
- Y1: ECS-2520MV-240-DN-TR -> YXC OT252024MJBA4SL (C669072). YXC
  datasheet: pin 1 tri-state enabled when floating (Y1 pin 1 is NC),
  pins 2/3/4 GND/OUT/VDD as on the ECS part, 1.8-3.3 V, same 2520
  land pattern.
- J2: Molex 0010897140 -> 0010897142 (C561778), same header and pin
  lengths with 15 uin instead of 30 uin gold (Mouser 538-10-89-7142).
- J8: Molex 0010897400 -> Wurth 61304021121 (C5364405, 732-5310-ND);
  insulator 0.25 mm taller.
- SW1/SW2: C&K PTS645VH58-2 LFS -> PTS645VK39-2 LFS (C285519,
  CKN10053-ND); footprints -> PTS645Vx39-2LFS (same pads as the
  Vx58/Vx31 ones used before).
- TUSB4041 kept; M2-M5 nuts fitted by hand.

Fields mirrored on the PCB footprints where the footprint does not
change. U16 and SW1/SW2 need F8 (Replace footprints); U16 then needs
re-routing. ERC unchanged at 342; DRC parity differs only by those
three footprint swaps.

Co-Authored-By: Claude Opus 5.5 <noreply@anthropic.com>
Parts:
- Y1: value ECS-2520MV-240-CN-TR -> OT252024MJBA4SL; Dist. P/N 50-ECS-2520MV-240-DN-TR-ND -> C669072; Distributor Digikey -> LCSC; LCSC (none) -> C669072; Manf. P/N ECS-2520MV-240-DN-TR -> OT252024MJBA4SL; Manufacturer ECS Inc. -> YXC; Part Description Oscillator, 24MHz, 1.6V~3.6V -> Oscillator, 24MHz, CMOS, 1.8V~3.3V, 20ppm, pin 1 enables wh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
Changed lines of the file:
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@@
 			)
 		)
-		(property "Value" "ECS-2520MV-240-CN-TR"
+		(property "Value" "OT252024MJBA4SL"
 			(at 177.546 169.418 0)
 			(show_name no)
@@
 			)
 		)
-		(property "Datasheet" "https://www.ecsxtal.com/store/pdf/ECS-2520MV.pdf"
+		(property "Datasheet" "https://www.lcsc.com/datasheet/lcsc_datasheet_2407310922_YXC-Crystal-Oscillators-OT252024MJBA4SL_C669072.pdf"
 			(at 156.845 156.845 0)
 			(hide yes)
@@
 			)
 		)
-		(property "Dist. P/N" "50-ECS-2520MV-240-DN-TR-ND"
+		(property "Dist. P/N" "C669072"
 			(at 161.29 160.02 0)
 			(hide yes)
@@
 			)
 		)
-		(property "Distributor" "Digikey"
+		(property "Distributor" "LCSC"
 			(at 161.29 160.02 0)
 			(hide yes)
@@
 			)
 		)
-		(property "Manf. P/N" "ECS-2520MV-240-DN-TR"
+		(property "Manf. P/N" "OT252024MJBA4SL"
 			(at 161.29 160.02 0)
 			(hide yes)
@@
 			)
 		)
-		(property "Manufacturer" "ECS Inc."
+		(property "LCSC" "C669072"
 			(at 161.29 160.02 0)
 			(hide yes)
@@
 			)
 		)
-		(property "Part Description" "Oscillator, 24MHz, 1.6V~3.6V"
+		(property "Manufacturer" "YXC"
 			(at 161.29 160.02 0)
 			(hide yes)
+			(show_name no)
+			(do_not_autoplace no)
+			(effects
+				(font
+					(size 1.27 1.27)
+				)
+			)
+		)
+		(property "Part Description" "Oscillator, 24MHz, CMOS, 1.8V~3.3V, 20ppm, pin 1 enables when open"
+			(at 161.29 160.02 0)
+			(hide yes)

Commit message: CM5 connectors: split Module1 into Module1 (pins 1-100) and Module2 (101-200)
Both Amphenol 10164227-1001A1RLF receptacles were one two-unit
symbol and one footprint with a single reference, which JLC's
placement file cannot express (one entry per part). Now:
- Symbols libreboard:ComputeModule5-CM5_A / _B (added to
  libreboard.kicad_sym), made from the two units of the old symbol
  with the same pins and pin positions, so every wire still lands.
  Module1 (CM5_GPIO sheet) keeps pins 1-100; the former unit B on
  CM5_HighSpeed becomes Module2 with pins 101-200 (pin numbers kept).
- Footprints libreboard:CM5_Connector_A / _B from the old
  Raspberry-Pi-5-Compute-Module footprint, origin at each connector
  centre (what JLC uses). A also carries the four CM5 mounting holes
  and the module outline; each keeps its own courtyard and 3D model.
- Board: the old footprint was replaced by the two new ones at the
  exact same pad positions (Module1 at 229.826/103.250, Module2 at
  195.826/103.250, both 180 deg), so tracks and vias are untouched.
  18 auto-named nets that embedded the old unit letter (e.g.
  Net-(Module1A-LED_nACT)) renamed on the board to the new names;
  Module2's reference text moved 1.5 mm off Module1's.

Checks: netlist connectivity identical pin for pin (1104 pins);
DRC with schematic parity, with and without zone refill, identical
to before (0 unconnected, same 104 warnings, same 11 parity items:
the old J11 four plus the U16/SW1/SW2 F8 still pending); ERC 342 ->
340 (the missing CM5IO library symbol warning is gone, the rest are
the same messages under the new reference). Placement export now
lists Module1 and Module2 at the connector centres.

Co-Authored-By: Claude Opus 5.5 <noreply@anthropic.com>
Parts:
- Module2: renamed from Module1; footprint libreboard:Raspberry-Pi-5-Compute-Module -> libreboard:CM5_Connector_B; symbol CM5IO:ComputeModule5-CM5 -> libreboard:ComputeModule5-CM5_B; Manf. P/N 10164227-1001A1RLF x2 -> 10164227-1001A1RLF
Changed lines of the file:
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@@
 	)
 	(symbol
-		(lib_id "CM5IO:ComputeModule5-CM5")
+		(lib_id "libreboard:ComputeModule5-CM5_B")
 		(at -71.12 86.36 0)
-		(unit 2)
+		(unit 1)
 		(body_style 1)
 		(exclude_from_sim no)
@@
 		(in_pos_files yes)
 		(dnp no)
-		(property "Reference" "Module1"
+		(property "Reference" "Module2"
 			(at 68.58 14.097 0)
 			(show_name no)
@@
 			)
 		)
-		(property "Footprint" "libreboard:Raspberry-Pi-5-Compute-Module"
+		(property "Footprint" "libreboard:CM5_Connector_B"
 			(at 71.12 113.03 0)
 			(hide yes)
@@
 			)
 		)
-		(property "Description" "RaspberryPi Compute module 5"
+		(property "Description" "Raspberry Pi Compute Module 5, connector B (pins 101-200)"
 			(at -71.12 86.36 0)
 			(hide yes)
@@
 			)
 		)
-		(property "Manf. P/N" "10164227-1001A1RLF x2"
+		(property "Manf. P/N" "10164227-1001A1RLF"
 			(at -71.12 86.36 0)
 			(hide yes)
@@
 				)
 			)
-		)
-		(pin "1"
-		)
-		(pin "10"
-		)
-		(pin "100"
-		)
-		(pin "11"
-		)
-		(pin "12"
-		)
-		(pin "13"
-		)
-		(pin "14"
-		)
-		(pin "15"
-		)
-		(pin "16"
-		)
-		(pin "17"
-		)
-		(pin "18"
-		)
-		(pin "19"
-		)
-		(pin "2"
-		)
-		(pin "20"
-		)
-		(pin "21"
-		)
-		(pin "22"
-		)
-		(pin "23"
-		)
-		(pin "24"
-		)
-		(pin "25"
-		)
-		(pin "26"
-		)
-		(pin "27"
-		)
-		(pin "28"
-		)
-		(pin "29"
-		)
-		(pin "3"
-		)
-		(pin "30"
-		)
-		(pin "31"
-		)
-		(pin "32"
-		)
-		(pin "33"
-		)
-		(pin "34"
-		)
-		(pin "35"
-		)
-		(pin "36"
-		)
-		(pin "37"
-		)
-		(pin "38"
-		)
-		(pin "39"
-		)
-		(pin "4"
-		)
-		(pin "40"
-		)
-		(pin "41"
-		)
-		(pin "42"
-		)
-		(pin "43"
-		)
-		(pin "44"
-		)
-		(pin "45"
-		)
-		(pin "46"
-		)
-		(pin "47"
-		)
-		(pin "48"
-		)
-		(pin "49"
-		)
-		(pin "5"
-		)
-		(pin "50"
-		)
-		(pin "51"
-		)
-		(pin "52"
-		)
-		(pin "53"
-		)
-		(pin "54"
-		)
-		(pin "55"
-		)
-		(pin "56"
-		)
-		(pin "57"
-		)
-		(pin "58"
-		)
-		(pin "59"
-		)
-		(pin "6"
-		)
-		(pin "60"
-		)
-		(pin "61"
-		)
-		(pin "62"
-		)
-		(pin "63"
-		)
-		(pin "64"
-		)
-		(pin "65"
-		)
-		(pin "66"
-		)
-		(pin "67"
-		)
-		(pin "68"
-		)
-		(pin "69"
-		)
-		(pin "7"
-		)
-		(pin "70"
-		)
-		(pin "71"
-		)
-		(pin "72"
-		)
-		(pin "73"
-		)
-		(pin "74"
-		)
-		(pin "75"
-		)
-		(pin "76"
-		)
-		(pin "77"
-		)
-		(pin "78"
-		)
-		(pin "79"
-		)
-		(pin "8"
-		)
-		(pin "80"
-		)
-		(pin "81"
-		)
-		(pin "82"
-		)
-		(pin "83"
-		)
-		(pin "84"
-		)
-		(pin "85"
-		)
-		(pin "86"
-		)
-		(pin "87"
-		)
-		(pin "88"
-		)
-		(pin "89"
-		)
-		(pin "9"
-		)
-		(pin "90"
-		)
-		(pin "91"
-		)
-		(pin "92"
-		)
-		(pin "93"
-		)
-		(pin "94"
-		)
-		(pin "95"
-		)
-		(pin "96"
-		)
-		(pin "97"
-		)
-		(pin "98"
-		)
-		(pin "99"
 		)
 		(pin "101"
@@
 			(project "libreboard"
 				(path "/e63e39d7-6ac0-4ffd-8aa3-1841a4541b55/00000000-0000-0000-0000-00005cff70b1"
-					(reference "Module1")
-					(unit 2)
-				)
-			)
+					(reference "Module2")
+					(unit 1)
+				)
+			)

Commit message: Freeze J11/J15/J7 symbols and J15 footprint in the project libraries
KiCad 10's stock library renamed the shield pin of
Connector:USB_C_Receptacle_USB2.0_16P (J11), USB_C_Receptacle (J15)
and Micro_SD_Card_Det2 (J7) from S1 / 11 to SH, and the stock
Connector_USB:USB_C_Receptacle_Molex_105450-0101 footprint now has SH
pads (and rounded pads). Our footprints use S1 / 11. Running "Update
symbols/footprints from library" would have left the shield pads of
these three connectors without their GND net.

- The three symbols, exactly as cached in the schematic, are now in
  libreboard.kicad_sym and the instances link there
  (libreboard:USB_C_Receptacle_USB2.0_16P, libreboard:USB_C_Receptacle,
  libreboard:Micro_SD_Card_Det2).
- J15's footprint, as placed on the board (28 pads, shields S1), is
  saved as libreboard:USB_C_Receptacle_Molex_105450-0101 and J15 links
  there in the schematic and on the board. J11 and J7 already used
  project footprints.

Netlist identical; ERC 333 -> 330 (the three lib_symbol_mismatch
warnings are gone); DRC with schematic parity unchanged.

Co-Authored-By: Claude Opus 5.5 <noreply@anthropic.com>
Parts:
- J15: footprint Connector_USB:USB_C_Receptacle_Molex_105450-0101 -> libreboard:USB_C_Receptacle_Molex_105450-0101; symbol Connector:USB_C_Receptacle -> libreboard:USB_C_Receptacle
Changed lines of the file:
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@@
 	)
 	(symbol
-		(lib_id "Connector:USB_C_Receptacle")
+		(lib_id "libreboard:USB_C_Receptacle")
 		(at 29.21 232.41 0)
 		(unit 1)
@@
 			)
 		)
-		(property "Footprint" "Connector_USB:USB_C_Receptacle_Molex_105450-0101"
+		(property "Footprint" "libreboard:USB_C_Receptacle_Molex_105450-0101"
 			(at 33.02 232.41 0)
 			(hide yes)

Commit message: BOM: J2 to a generic 2x7 header, J22 to the EDAC HDMI connector
JLC has no footprint for the Molex parts chosen before (C561778,
C5240402), so its preview could not show or place them.

- J2: BOOMELE 2.54-2*7P (C71397, gold, 21.5k at JLC). 6/3 mm pins and a
  2.5 mm insulator instead of the C-Grid's 6.1/2.8 mm and 2.29 mm.
- J22: EDAC 690-019-298-412 (C5291558, 1,850 at JLC), the part the
  footprint from Raspberry Pi's CM5 IO board was drawn for.

JLC's footprints for both match ours pad for pad. Neither part is at
DigiKey or Mouser, so Distributor = LCSC. Fields only: ERC (330) and DRC
with schematic parity (103, 4 parity) unchanged.

Co-Authored-By: Claude Opus 5.5 <noreply@anthropic.com>
Parts:
- J22: Dist. P/N 900-2086581051TR-ND -> C5291558; Distributor Digikey -> LCSC; LCSC C5240402 -> C5291558; Manf. P/N 2086581051 -> 690-019-298-412; Manufacturer Molex -> EDAC; Part Description Connector, HDMI 2.1, Female, Right Angle, 19 pin, SMD -> Connector, HDMI Type A, Female, Right Angle, 19 pin, SMD
Changed lines of the file:
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@@
 			)
 		)
-		(property "Datasheet" "https://www.molex.com/en-us/products/part-detail-pdf/2086581051?display=pdf"
+		(property "Datasheet" ""
 			(at 264.795 50.8 0)
 			(hide yes)
@@
 			)
 		)
-		(property "Part Description" "Connector, HDMI 2.1, Female, Right Angle, 19 pin, SMD"
+		(property "Part Description" "Connector, HDMI Type A, Female, Right Angle, 19 pin, SMD"
 			(at 264.16 50.8 0)
 			(hide yes)
@@
 			)
 		)
-		(property "Dist. P/N" "900-2086581051TR-ND"
+		(property "Dist. P/N" "C5291558"
 			(at 264.16 50.8 0)
 			(hide yes)
@@
 			)
 		)
-		(property "Distributor" "Digikey"
+		(property "Distributor" "LCSC"
 			(at 264.16 50.8 0)
 			(hide yes)
@@
 			)
 		)
-		(property "Manf. P/N" "2086581051"
+		(property "Manf. P/N" "690-019-298-412"
 			(at 264.16 50.8 0)
 			(hide yes)
@@
 			)
 		)
-		(property "Manufacturer" "Molex"
+		(property "Manufacturer" "EDAC"
 			(at 264.16 50.8 0)
 			(hide yes)
@@
 			)
 		)
-		(property "LCSC" "C5240402"
+		(property "LCSC" "C5291558"
 			(at 264.16 50.8 0)
 			(hide yes)

Commit message: BOM: Y1 to Epson X1G0041710031 (SG-210STF 24 MHz)
JLC's stock of the YXC OT252024MJBA4SL (C669072) fell from 4,530 to 1.
The Epson part (C70559, 7,235 at JLC) has the same pinout: pin 1 = ST,
output running when high or open (Y1 pin 1 is unconnected), 2 GND,
3 OUT, 4 VCC; 1.6-3.6 V supply (+1V8), CMOS, +-50 ppm, start-up <= 3 ms.
JLC's footprint is the same as for the YXC part and matches ours.
Fields only: ERC, DRC and schematic parity unchanged.

Refs #24

Co-Authored-By: Claude Opus 5.5 <noreply@anthropic.com>
Parts:
- Y1: value OT252024MJBA4SL -> X1G0041710031; Dist. P/N C669072 -> C70559; LCSC C669072 -> C70559; Manf. P/N OT252024MJBA4SL -> X1G0041710031; Manufacturer YXC -> Seiko Epson; Part Description Oscillator, 24MHz, CMOS, 1.8V~3.3V, 20ppm, pin 1 enables wh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 -> Oscillator SG-210STF, 24MHz, CMOS, 1.6V~3.6V, 50ppm, pin 1 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
Changed lines of the file:
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@@
 			)
 		)
-		(property "Value" "OT252024MJBA4SL"
+		(property "Value" "X1G0041710031"
 			(at 177.546 169.418 0)
 			(show_name no)
@@
 			)
 		)
-		(property "Datasheet" "https://www.lcsc.com/datasheet/lcsc_datasheet_2407310922_YXC-Crystal-Oscillators-OT252024MJBA4SL_C669072.pdf"
+		(property "Datasheet" "https://www.lcsc.com/datasheet/lcsc_datasheet_2404171436_Seiko-Epson-X1G0041710031_C70559.pdf"
 			(at 156.845 156.845 0)
 			(hide yes)
@@
 			)
 		)
-		(property "Dist. P/N" "C669072"
+		(property "Dist. P/N" "C70559"
 			(at 161.29 160.02 0)
 			(hide yes)
@@
 			)
 		)
-		(property "Manf. P/N" "OT252024MJBA4SL"
+		(property "Manf. P/N" "X1G0041710031"
 			(at 161.29 160.02 0)
 			(hide yes)
@@
 			)
 		)
-		(property "LCSC" "C669072"
+		(property "LCSC" "C70559"
 			(at 161.29 160.02 0)
 			(hide yes)
@@
 			)
 		)
-		(property "Manufacturer" "YXC"
+		(property "Manufacturer" "Seiko Epson"
 			(at 161.29 160.02 0)
 			(hide yes)
@@
 			)
 		)
-		(property "Part Description" "Oscillator, 24MHz, CMOS, 1.8V~3.3V, 20ppm, pin 1 enables when open"
+		(property "Part Description" "Oscillator SG-210STF, 24MHz, CMOS, 1.6V~3.6V, 50ppm, pin 1 (ST) runs when open"
 			(at 161.29 160.02 0)
 			(hide yes)
