File: CM5_GPIO.kicad_sch (KiCad schematic)
At the start: 42 parts, among them J14 JST_BM04B-SRSS-TB, J16 JST_BM04B-SRSS-TB, J19 Conn_1x03_Male, J2 Conn_2x07_Male, J3 Conn_1x03_Male, J7 Micro_SD_Card_Det, J8 Conn_2x20_Male, SW1 Right angle Tact button, SW2 Right angle Tact button, U1 TPD4EUSB30, U16 SN74AHCT1G125DRLR, U17 TCA9538DBR, U18 RT9742GGJ5, U2 TPD4EUSB30, U3 MagJack-A70-112-331N126, U5 74LVC1G07SE-7, U9 SK6812

Commit message: switch C21 and C52 to 50V, 0805 size and reposition; Rev2 text
Parts:
- BT1: Dist. P/N (none) -> 343-BAT-HLD-007-SMT-TR-ND; Distributor (none) -> Digikey; Manf. P/N (none) -> BAT-HLD-007-SMT-TR; Manufacturer (none) -> TE Connectivity Linx; Part Description Battery Retainer Coin, 20.0mm 1 Cell SMD (SMT) Tab -> BATTERY RETAINER COIN 12.5MM SMD
Changed lines of the file:
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@@
 			)
 		)
-		(property "Datasheet" ""
+		(property "Datasheet" "https://www.te.com/commerce/DocumentDelivery/DDEController?Action=srchrtrv&DocNm=BAT-HLD-007-SMT-TR&DocType=Data+Sheet&DocLang=English&DocFormat=pdf&PartCntxt=BAT-HLD-007-SMT-TR"
 			(at 201.93 175.26 0)
 			(effects
@@
 			)
 		)
-		(property "Part Description" "	Battery Retainer Coin, 20.0mm 1 Cell SMD (SMT) Tab"
+		(property "Part Description" "BATTERY RETAINER COIN 12.5MM SMD"
 			(at 201.93 175.26 0)
 			(effects
@@
 				(hide yes)
 			)
+		)
+		(property "Dist. P/N" "343-BAT-HLD-007-SMT-TR-ND"
+			(at 201.93 175.26 0)
+			(effects
+				(font
+					(size 1.27 1.27)
+				)
+				(hide yes)
+			)
+		)
+		(property "Distributor" "Digikey"
+			(at 201.93 175.26 0)
+			(effects
+				(font
+					(size 1.27 1.27)
+				)
+				(hide yes)
+			)
+		)
+		(property "Manf. P/N" "BAT-HLD-007-SMT-TR"
+			(at 201.93 175.26 0)
+			(effects
+				(font
+					(size 1.27 1.27)
+				)
+				(hide yes)
+			)
+		)
+		(property "Manufacturer" "TE Connectivity Linx"
+			(at 201.93 175.26 0)
+			(effects
+				(font
+					(size 1.27 1.27)
+				)
+				(hide yes)
+			)
