File: CM5_GPIO.kicad_sch (KiCad schematic)
At the start: 43 parts, among them J14 JST_BM04B-SRSS-TB, J16 JST_BM04B-SRSS-TB, J19 Conn_1x03_Male, J2 Conn_2x07_Male, J3 Conn_1x03_Male, J7 Micro_SD_Card_Det, J8 Conn_2x20_Male, SW1 Right angle Tact button, SW2 Right angle Tact button, U1 TPD4EUSB30, U16 SN74AHCT1G125DRLR, U17 TCA9538DBR, U18 RT9742GGJ5, U2 TPD4EUSB30, U3 MagJack-A70-112-331N126, U5 74LVC1G07SE-7, U9 SK6812

Commit message: U3: MagJack TMJG4926HENL -> LINK-PP LPJG0926HENL (same pinout)
The Rev1 Ethernet fault was never a broken winding: the jacks fitted
(and the spares) are Taoglas TMJG0813GENL, which fits the same holes
but has a different pinout (4/5 = a signal pair, 9 = centre tap,
10 = GND, no pins 11-14). On our footprint that shorts one pair on
the CT net and puts TRD3 on the centre tap and ground, so 100 Mb/s
works and gigabit never can.

U3 now names LINK-PP LPJG0926HENL. Its datasheet (LP18022610 rev A)
has the same schematic, pin layout and footprint as TMJG4926HENL
(SPE-23-8-193-B): TD1-TD4 on 1/2, 3/6, 7/8, 9/10, CT 4/5, VC 11-14,
green LED 15/16, yellow 17/18. JLC C22457393, 2305 in stock; the
Taoglas part has 0 at JLC and 4 at DigiKey. Rated 0-70 C instead of
-40-85 C. Not found at DigiKey or Mouser, so Distributor = LCSC
(same convention as U9).

Fields changed on the symbol and the PCB footprint: Value,
Datasheet, Manufacturer, Manf. P/N, Distributor, Dist. P/N, LCSC,
and a Description note not to substitute TMJG0813GENL. Sourcing
report updated to match.

ERC 342 unchanged; DRC with schematic parity unchanged.

Co-Authored-By: Claude Opus 5.5 <noreply@anthropic.com>
Parts:
- U3: value MagJack-A70-112-331N126 -> LPJG0926HENL; Dist. P/N 931-TMJG4926HENL-ND -> C22457393; Distributor Digikey -> LCSC; LCSC C37415176 -> C22457393; Manf. P/N TMJG4926HENL -> LPJG0926HENL; Manufacturer Taoglas Limited -> LINK-PP
Changed lines of the file:
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@@
 			)
 		)
-		(property "Value" "MagJack-A70-112-331N126"
+		(property "Value" "LPJG0926HENL"
 			(at 250.19 92.71 0)
 			(show_name no)
@@
 			)
 		)
-		(property "Datasheet" "https://www.taoglas.com/datasheets/TMJG4926HENL.pdf"
+		(property "Datasheet" "https://www.l-p.com/file/datasheet/lpjg0926henl.pdf"
 			(at 267.97 92.71 0)
 			(hide yes)
@@
 			)
 		)
-		(property "Description" ""
+		(property "Description" "RJ45 1G MagJack, LPJG0926HENL/TMJG4926HENL pinout (4,5 = CT; 9,10 = TD4; 11-14 = VC). Do not substitute TMJG0813GENL: different pinout (9 = CT, 10 = GND)."
 			(at 267.97 92.71 0)
 			(hide yes)
@@
 			)
 		)
-		(property "Dist. P/N" "931-TMJG4926HENL-ND"
+		(property "Dist. P/N" "C22457393"
 			(at 267.97 92.71 0)
 			(hide yes)
@@
 			)
 		)
-		(property "Distributor" "Digikey"
+		(property "Distributor" "LCSC"
 			(at 267.97 92.71 0)
 			(hide yes)
@@
 			)
 		)
-		(property "Manf. P/N" "TMJG4926HENL"
+		(property "Manf. P/N" "LPJG0926HENL"
 			(at 267.97 92.71 0)
 			(hide yes)
@@
 			)
 		)
-		(property "Manufacturer" "Taoglas Limited"
+		(property "Manufacturer" "LINK-PP"
 			(at 267.97 92.71 0)
 			(hide yes)
@@
 			)
 		)
-		(property "LCSC" "C37415176"
+		(property "LCSC" "C22457393"
 			(at 267.97 92.71 0)
 			(hide yes)

Commit message: Ethernet TVS U1/U2 (TPD4EUSB30): not fitted (DNP)
They come from the CM5 IO board, whose schematic labels them
"Ethernet POE Protection": there the cable-side centre taps go to a
PoE header (J9). LibreBoard has no PoE (TR0-3_TAP unconnected) and
the MagJack already isolates the cable side (1500 Vrms). On Rev1 the
hand-soldered U1/U2 were the cause of the 100 Mb/s link drops, and
the board ran clean with them removed.

The footprints stay (flow-through: pin 1 to 10, 2 to 9, 4 to 7,
5 to 6 under the package), so the lines are continuous with them
empty and they can be fitted later. Same convention as C26: still in
the BOM, dnp on the symbol and on the footprint.

ERC 342 unchanged; DRC with schematic parity unchanged. With
--exclude-dnp, U1/U2 drop out of the BOM and placement exports.
Sourcing report: notes, and setup-fee count 61 -> 60.

Co-Authored-By: Claude Opus 5.5 <noreply@anthropic.com>
Parts:
- U1, U2: now not fitted
Changed lines of the file:
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@@
 		(on_board yes)
 		(in_pos_files yes)
-		(dnp no)
+		(dnp yes)
 		(property "Reference" "U2"
 			(at 207.01 50.3682 0)
@@
 		(on_board yes)
 		(in_pos_files yes)
-		(dnp no)
+		(dnp yes)
 		(property "Reference" "U1"
 			(at 207.01 18.6182 0)

Commit message: BOM: JLC sourcing decisions (U4/U14, U16, U17, BT1, Y1, J2, J8, SW1/SW2)
Michael's decisions on bom/rev3-sourcing.md section 1:
- U4/U14: TPS552892RYQR (unobtainable) -> TPS552892QWRYQRQ1, the
  AEC-Q100 version (same pins, RYQ package, VREF, input range).
  To be bought at Mouser and supplied to JLC (JLC and DigiKey 0).
- U16: SOT-553 DRLR (0 at JLC) -> SC-70-5 SN74AHCT1G125DCKR
  (C350557), same pinout; SC-70-5 because U16 is 1.5-2.3 mm from
  C71/C70/R9/R52. Footprint Package_TO_SOT_SMD:SOT-353_SC-70-5.
- U17 TCA9538DBR: hand-fitted from DigiKey; in_pos_files no /
  exclude_from_pos_files.
- BT1: Linx BAT-HLD-007-SMT-TR -> Keystone 3000TR (C6997853), the
  12 mm retainer it copies: + tabs at +-7.9 mm, - is the board pad,
  so the footprint stays.
- Y1: ECS-2520MV-240-DN-TR -> YXC OT252024MJBA4SL (C669072). YXC
  datasheet: pin 1 tri-state enabled when floating (Y1 pin 1 is NC),
  pins 2/3/4 GND/OUT/VDD as on the ECS part, 1.8-3.3 V, same 2520
  land pattern.
- J2: Molex 0010897140 -> 0010897142 (C561778), same header and pin
  lengths with 15 uin instead of 30 uin gold (Mouser 538-10-89-7142).
- J8: Molex 0010897400 -> Wurth 61304021121 (C5364405, 732-5310-ND);
  insulator 0.25 mm taller.
- SW1/SW2: C&K PTS645VH58-2 LFS -> PTS645VK39-2 LFS (C285519,
  CKN10053-ND); footprints -> PTS645Vx39-2LFS (same pads as the
  Vx58/Vx31 ones used before).
- TUSB4041 kept; M2-M5 nuts fitted by hand.

Fields mirrored on the PCB footprints where the footprint does not
change. U16 and SW1/SW2 need F8 (Replace footprints); U16 then needs
re-routing. ERC unchanged at 342; DRC parity differs only by those
three footprint swaps.

Co-Authored-By: Claude Opus 5.5 <noreply@anthropic.com>
Parts:
- BT1: Dist. P/N 343-BAT-HLD-007-SMT-TR-ND -> 36-3000TR-ND; LCSC C7219081 -> C6997853; Manf. P/N BAT-HLD-007-SMT-TR -> 3000TR; Manufacturer TE Connectivity Linx -> Keystone Electronics; Part Description BATTERY RETAINER COIN 12.5MM SMD -> BATTERY RETAINER COIN 12MM SMD (CR1216/1220/1225)
- J2: Dist. P/N WM9875-ND -> 538-10-89-7142; Distributor Digikey -> Mouser; LCSC (none) -> C561778; Manf. P/N 0010897140 -> 0010897142; Part Description Pin Header, Male, 2x07, 2.54mm P, Vertical -> Pin Header, Male, 2x07, 2.54mm P, Vertical, 15 uin gold
- J8: Dist. P/N WM19411-ND -> 732-5310-ND; LCSC (none) -> C5364405; Manf. P/N 0010897400 -> 61304021121; Manufacturer Molex -> Wurth Elektronik; Part Description Pin Header, Male, 2x20, 2.54mm P, Vertical -> Pin Header, Male, 2x20, 2.54mm P, Vertical, 2.54mm insulator
- SW1: footprint Button_Switch_THT:SW_Tactile_SPST_Angled_PTS645Vx58-2LFS -> Button_Switch_THT:SW_Tactile_SPST_Angled_PTS645Vx39-2LFS; Dist. P/N CKN9120-ND -> CKN10053-ND; LCSC (none) -> C285519; Manf. P/N PTS645VH58-2 LFS -> PTS645VK39-2 LFS
- SW2: footprint Button_Switch_THT:SW_Tactile_SPST_Angled_PTS645Vx31-2LFS -> Button_Switch_THT:SW_Tactile_SPST_Angled_PTS645Vx39-2LFS; Dist. P/N CKN9120-ND -> CKN10053-ND; LCSC (none) -> C285519; Manf. P/N PTS645VH58-2 LFS -> PTS645VK39-2 LFS
- U16: value SN74AHCT1G125DRLR -> SN74AHCT1G125DCKR; footprint libreboard:DRL5-L -> Package_TO_SOT_SMD:SOT-353_SC-70-5; Dist. P/N 296-19379-2-ND -> C350557; Distributor Digikey -> LCSC; LCSC C507216 -> C350557; Manf. P/N SN74AHCT1G125DRLR -> SN74AHCT1G125DCKR; Part Description Buffer, Non-Inverting 1 Element 1 Bit per Element 3-State Output SOT-5 -> Buffer, Non-Inverting 1 Element 1 Bit per Element 3-State Output SC-70-5
Changed lines of the file:
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@@
 			)
 		)
-		(property "Datasheet" ""
+		(property "Datasheet" "https://www.we-online.com/catalog/datasheet/61304021121.pdf"
 			(at 157.48 46.99 0)
 			(hide yes)
@@
 			)
 		)
-		(property "Part Description" "Pin Header, Male, 2x20, 2.54mm P, Vertical"
+		(property "Part Description" "Pin Header, Male, 2x20, 2.54mm P, Vertical, 2.54mm insulator"
 			(at 157.48 46.99 0)
 			(hide yes)
@@
 			)
 		)
-		(property "Dist. P/N" "WM19411-ND"
+		(property "Dist. P/N" "732-5310-ND"
 			(at 157.48 46.99 0)
 			(hide yes)
@@
 			)
 		)
-		(property "Manf. P/N" "0010897400"
+		(property "Manf. P/N" "61304021121"
 			(at 157.48 46.99 0)
 			(hide yes)
@@
 			)
 		)
-		(property "Manufacturer" "Molex"
+		(property "LCSC" "C5364405"
+			(at 157.48 46.99 0)
+			(hide yes)
+			(show_name no)
+			(do_not_autoplace no)
+			(effects
+				(font
+					(size 1.27 1.27)
+				)
+			)
+		)
+		(property "Manufacturer" "Wurth Elektronik"
 			(at 157.48 46.99 0)
 			(hide yes)
@@
 			)
 		)
-		(property "Part Description" "Pin Header, Male, 2x07, 2.54mm P, Vertical"
+		(property "Part Description" "Pin Header, Male, 2x07, 2.54mm P, Vertical, 15 uin gold"
 			(at 36.83 177.8 0)
 			(hide yes)
@@
 			)
 		)
-		(property "Dist. P/N" "WM9875-ND"
+		(property "Dist. P/N" "538-10-89-7142"
 			(at 36.83 177.8 0)
 			(hide yes)
@@
 			)
 		)
-		(property "Distributor" "Digikey"
+		(property "Distributor" "Mouser"
 			(at 36.83 177.8 0)
 			(hide yes)
@@
 			)
 		)
-		(property "Manf. P/N" "0010897140"
+		(property "Manf. P/N" "0010897142"
+			(at 36.83 177.8 0)
+			(hide yes)
+			(show_name no)
+			(do_not_autoplace no)
+			(effects
+				(font
+					(size 1.27 1.27)
+				)
+			)
+		)
+		(property "LCSC" "C561778"
 			(at 36.83 177.8 0)
 			(hide yes)
@@
 			)
 		)
-		(property "Datasheet" "https://www.te.com/commerce/DocumentDelivery/DDEController?Action=srchrtrv&DocNm=BAT-HLD-007-SMT-TR&DocType=Data+Sheet&DocLang=English&DocFormat=pdf&PartCntxt=BAT-HLD-007-SMT-TR"
+		(property "Datasheet" "https://www.keyelco.com/userAssets/file/K75p11.pdf"
 			(at 201.93 175.26 0)
 			(hide yes)
@@
 			)
 		)
-		(property "Part Description" "BATTERY RETAINER COIN 12.5MM SMD"
+		(property "Part Description" "BATTERY RETAINER COIN 12MM SMD (CR1216/1220/1225)"
 			(at 201.93 175.26 0)
 			(hide yes)
@@
 			)
 		)
-		(property "Dist. P/N" "343-BAT-HLD-007-SMT-TR-ND"
+		(property "Dist. P/N" "36-3000TR-ND"
 			(at 201.93 175.26 0)
 			(hide yes)
@@
 			)
 		)
-		(property "Manf. P/N" "BAT-HLD-007-SMT-TR"
+		(property "Manf. P/N" "3000TR"
 			(at 201.93 175.26 0)
 			(hide yes)
@@
 			)
 		)
-		(property "Manufacturer" "TE Connectivity Linx"
+		(property "Manufacturer" "Keystone Electronics"
 			(at 201.93 175.26 0)
 			(hide yes)
@@
 			)
 		)
-		(property "LCSC" "C7219081"
+		(property "LCSC" "C6997853"
 			(at 201.93 175.26 0)
 			(hide yes)
@@
 			)
 		)
-		(property "Value" "SN74AHCT1G125DRLR"
+		(property "Value" "SN74AHCT1G125DCKR"
 			(at 129.032 236.474 0)
 			(show_name no)
@@
 			)
 		)
-		(property "Footprint" "libreboard:DRL5-L"
+		(property "Footprint" "Package_TO_SOT_SMD:SOT-353_SC-70-5"
 			(at 87.63 243.84 0)
 			(hide yes)
@@
 			)
 		)
-		(property "Dist. P/N" "296-19379-2-ND"
+		(property "Dist. P/N" "C350557"
 			(at 87.63 243.84 0)
 			(hide yes)
@@
 			)
 		)
-		(property "Distributor" "Digikey"
+		(property "Distributor" "LCSC"
 			(at 87.63 243.84 0)
 			(hide yes)
@@
 			)
 		)
-		(property "Manf. P/N" "SN74AHCT1G125DRLR"
+		(property "Manf. P/N" "SN74AHCT1G125DCKR"
 			(at 87.63 243.84 0)
 			(hide yes)
@@
 			)
 		)
-		(property "Part Description" "Buffer, Non-Inverting 1 Element 1 Bit per Element 3-State Output SOT-5"
+		(property "Part Description" "Buffer, Non-Inverting 1 Element 1 Bit per Element 3-State Output SC-70-5"
 			(at 87.63 243.84 0)
 			(hide yes)
@@
 			)
 		)
-		(property "LCSC" "C507216"
+		(property "LCSC" "C350557"
 			(at 87.63 243.84 0)
 			(hide yes)
@@
 			)
 		)
-		(property "Footprint" "Button_Switch_THT:SW_Tactile_SPST_Angled_PTS645Vx58-2LFS"
+		(property "Footprint" "Button_Switch_THT:SW_Tactile_SPST_Angled_PTS645Vx39-2LFS"
 			(at 82.55 180.34 0)
 			(hide yes)
@@
 			)
 		)
-		(property "Datasheet" ""
+		(property "Datasheet" "https://www.littelfuse.com/assetdocs/littelfuse-c-k-tactile-pts645v-series-datasheet?assetguid=5014fb06-c6ac-482c-8b16-1ea09e49f7c0"
 			(at 82.55 180.34 0)
 			(hide yes)
@@
 			)
 		)
-		(property "Dist. P/N" "CKN9120-ND"
+		(property "Dist. P/N" "CKN10053-ND"
 			(at 77.47 180.34 90)
 			(hide yes)
@@
 			)
 		)
-		(property "Manf. P/N" "PTS645VH58-2 LFS"
+		(property "Manf. P/N" "PTS645VK39-2 LFS"
+			(at 77.47 180.34 90)
+			(hide yes)
+			(show_name no)
+			(do_not_autoplace no)
+			(effects
+				(font
+					(size 1.27 1.27)
+				)
+			)
+		)
+		(property "LCSC" "C285519"
 			(at 77.47 180.34 90)
 			(hide yes)
@@
 			)
 		)
-		(property "Footprint" "Button_Switch_THT:SW_Tactile_SPST_Angled_PTS645Vx31-2LFS"
+		(property "Footprint" "Button_Switch_THT:SW_Tactile_SPST_Angled_PTS645Vx39-2LFS"
 			(at 81.28 158.75 0)
 			(hide yes)
@@
 			)
 		)
-		(property "Datasheet" ""
+		(property "Datasheet" "https://www.littelfuse.com/assetdocs/littelfuse-c-k-tactile-pts645v-series-datasheet?assetguid=5014fb06-c6ac-482c-8b16-1ea09e49f7c0"
 			(at 81.28 158.75 0)
 			(hide yes)
@@
 			)
 		)
-		(property "Dist. P/N" "CKN9120-ND"
+		(property "Dist. P/N" "CKN10053-ND"
 			(at 76.2 158.75 90)
 			(hide yes)
@@
 			)
 		)
-		(property "Manf. P/N" "PTS645VH58-2 LFS"
+		(property "Manf. P/N" "PTS645VK39-2 LFS"
+			(at 76.2 158.75 90)
+			(hide yes)
+			(show_name no)
+			(do_not_autoplace no)
+			(effects
+				(font
+					(size 1.27 1.27)
+				)
+			)
+		)
+		(property "LCSC" "C285519"
 			(at 76.2 158.75 90)
 			(hide yes)
@@
 		(in_bom yes)
 		(on_board yes)
-		(in_pos_files yes)
+		(in_pos_files no)
 		(dnp no)
 		(fields_autoplaced yes)
@@
 			)
 		)
-		(property "Description" ""
+		(property "Description" "Hand-fitted after JLC assembly (JLC stock too low); excluded from the placement file."
 			(at 72.39 236.22 0)
 			(hide yes)

Commit message: CM5 connectors: split Module1 into Module1 (pins 1-100) and Module2 (101-200)
Both Amphenol 10164227-1001A1RLF receptacles were one two-unit
symbol and one footprint with a single reference, which JLC's
placement file cannot express (one entry per part). Now:
- Symbols libreboard:ComputeModule5-CM5_A / _B (added to
  libreboard.kicad_sym), made from the two units of the old symbol
  with the same pins and pin positions, so every wire still lands.
  Module1 (CM5_GPIO sheet) keeps pins 1-100; the former unit B on
  CM5_HighSpeed becomes Module2 with pins 101-200 (pin numbers kept).
- Footprints libreboard:CM5_Connector_A / _B from the old
  Raspberry-Pi-5-Compute-Module footprint, origin at each connector
  centre (what JLC uses). A also carries the four CM5 mounting holes
  and the module outline; each keeps its own courtyard and 3D model.
- Board: the old footprint was replaced by the two new ones at the
  exact same pad positions (Module1 at 229.826/103.250, Module2 at
  195.826/103.250, both 180 deg), so tracks and vias are untouched.
  18 auto-named nets that embedded the old unit letter (e.g.
  Net-(Module1A-LED_nACT)) renamed on the board to the new names;
  Module2's reference text moved 1.5 mm off Module1's.

Checks: netlist connectivity identical pin for pin (1104 pins);
DRC with schematic parity, with and without zone refill, identical
to before (0 unconnected, same 104 warnings, same 11 parity items:
the old J11 four plus the U16/SW1/SW2 F8 still pending); ERC 342 ->
340 (the missing CM5IO library symbol warning is gone, the rest are
the same messages under the new reference). Placement export now
lists Module1 and Module2 at the connector centres.

Co-Authored-By: Claude Opus 5.5 <noreply@anthropic.com>
Parts:
- Module1: footprint libreboard:Raspberry-Pi-5-Compute-Module -> libreboard:CM5_Connector_A; symbol CM5IO:ComputeModule5-CM5 -> libreboard:ComputeModule5-CM5_A; Manf. P/N 10164227-1001A1RLF x2 -> 10164227-1001A1RLF
Changed lines of the file:
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@@
 	)
 	(symbol
-		(lib_id "CM5IO:ComputeModule5-CM5")
+		(lib_id "libreboard:ComputeModule5-CM5_A")
 		(at 72.39 77.47 0)
 		(unit 1)
@@
 			)
 		)
-		(property "Footprint" "libreboard:Raspberry-Pi-5-Compute-Module"
+		(property "Footprint" "libreboard:CM5_Connector_A"
 			(at 214.63 104.14 0)
 			(hide yes)
@@
 			)
 		)
-		(property "Description" "RaspberryPi Compute module 5"
+		(property "Description" "Raspberry Pi Compute Module 5, connector A (pins 1-100)"
 			(at 72.39 77.47 0)
 			(hide yes)
@@
 			)
 		)
-		(property "Manf. P/N" "10164227-1001A1RLF x2"
+		(property "Manf. P/N" "10164227-1001A1RLF"
 			(at 72.39 77.47 0)
 			(hide yes)
@@
 		(pin "99"
 		)
-		(pin "101"
-		)
-		(pin "102"
-		)
-		(pin "103"
-		)
-		(pin "104"
-		)
-		(pin "105"
-		)
-		(pin "106"
-		)
-		(pin "107"
-		)
-		(pin "108"
-		)
-		(pin "109"
-		)
-		(pin "110"
-		)
-		(pin "111"
-		)
-		(pin "112"
-		)
-		(pin "113"
-		)
-		(pin "114"
-		)
-		(pin "115"
-		)
-		(pin "116"
-		)
-		(pin "117"
-		)
-		(pin "118"
-		)
-		(pin "119"
-		)
-		(pin "120"
-		)
-		(pin "121"
-		)
-		(pin "122"
-		)
-		(pin "123"
-		)
-		(pin "124"
-		)
-		(pin "125"
-		)
-		(pin "126"
-		)
-		(pin "127"
-		)
-		(pin "128"
-		)
-		(pin "129"
-		)
-		(pin "130"
-		)
-		(pin "131"
-		)
-		(pin "132"
-		)
-		(pin "133"
-		)
-		(pin "134"
-		)
-		(pin "135"
-		)
-		(pin "136"
-		)
-		(pin "137"
-		)
-		(pin "138"
-		)
-		(pin "139"
-		)
-		(pin "140"
-		)
-		(pin "141"
-		)
-		(pin "142"
-		)
-		(pin "143"
-		)
-		(pin "144"
-		)
-		(pin "145"
-		)
-		(pin "146"
-		)
-		(pin "147"
-		)
-		(pin "148"
-		)
-		(pin "149"
-		)
-		(pin "150"
-		)
-		(pin "151"
-		)
-		(pin "152"
-		)
-		(pin "153"
-		)
-		(pin "154"
-		)
-		(pin "155"
-		)
-		(pin "156"
-		)
-		(pin "157"
-		)
-		(pin "158"
-		)
-		(pin "159"
-		)
-		(pin "160"
-		)
-		(pin "161"
-		)
-		(pin "162"
-		)
-		(pin "163"
-		)
-		(pin "164"
-		)
-		(pin "165"
-		)
-		(pin "166"
-		)
-		(pin "167"
-		)
-		(pin "168"
-		)
-		(pin "169"
-		)
-		(pin "170"
-		)
-		(pin "171"
-		)
-		(pin "172"
-		)
-		(pin "173"
-		)
-		(pin "174"
-		)
-		(pin "175"
-		)
-		(pin "176"
-		)
-		(pin "177"
-		)
-		(pin "178"
-		)
-		(pin "179"
-		)
-		(pin "180"
-		)
-		(pin "181"
-		)
-		(pin "182"
-		)
-		(pin "183"
-		)
-		(pin "184"
-		)
-		(pin "185"
-		)
-		(pin "186"
-		)
-		(pin "187"
-		)
-		(pin "188"
-		)
-		(pin "189"
-		)
-		(pin "190"
-		)
-		(pin "191"
-		)
-		(pin "192"
-		)
-		(pin "193"
-		)
-		(pin "194"
-		)
-		(pin "195"
-		)
-		(pin "196"
-		)
-		(pin "197"
-		)
-		(pin "198"
-		)
-		(pin "199"
-		)
-		(pin "200"
-		)
 		(instances

Commit message: Fan controller: 10k pull-up on unused TACH5; ERC drawing cleanup
From the ERC review (342 messages, none an electrical fault):
- U10 (EMC2305) TACH5, pin 16, was floating. The datasheet types the
  TACH inputs as open-drain inputs that need an external pull-up, so
  it gets the same 10k to +3.3v as TACH1-4: new R64 (ERJ-U02F1002X,
  LCSC C25744) above R21-R24 on the +3.3v bus, joined to pin 16 by a
  TACH5 label. No-connect flags on the unused PWM5 (pin 15) and
  ALERT# (pin 12) outputs.
- Removed the two GPIO_VREF sheet pins on the root sheet and the wire
  between them: neither sub-sheet has that label and the wire joined
  only those two pins. The CM5's GPIO_VREF pin is on +3.3v inside
  CM5_GPIO as before.
- Removed a no-connect flag in CM5_GPIO at (185.42, 118.11) that has
  never been on a pin.

Netlist: only R64 (+3.3v / TACH5) and U10 pin 16 (-> TACH5) change.
ERC 340 -> 333. PCB needs F8 to add R64 (0402) near U10, plus routing.

Co-Authored-By: Claude Opus 5.5 <noreply@anthropic.com>
Connections:
- no-connect marks 11 -> 10
Changed lines of the file:
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@@
-	)
-	(no_connect
-		(at 185.42 118.11)
 	)
 	(no_connect

Commit message: Freeze J11/J15/J7 symbols and J15 footprint in the project libraries
KiCad 10's stock library renamed the shield pin of
Connector:USB_C_Receptacle_USB2.0_16P (J11), USB_C_Receptacle (J15)
and Micro_SD_Card_Det2 (J7) from S1 / 11 to SH, and the stock
Connector_USB:USB_C_Receptacle_Molex_105450-0101 footprint now has SH
pads (and rounded pads). Our footprints use S1 / 11. Running "Update
symbols/footprints from library" would have left the shield pads of
these three connectors without their GND net.

- The three symbols, exactly as cached in the schematic, are now in
  libreboard.kicad_sym and the instances link there
  (libreboard:USB_C_Receptacle_USB2.0_16P, libreboard:USB_C_Receptacle,
  libreboard:Micro_SD_Card_Det2).
- J15's footprint, as placed on the board (28 pads, shields S1), is
  saved as libreboard:USB_C_Receptacle_Molex_105450-0101 and J15 links
  there in the schematic and on the board. J11 and J7 already used
  project footprints.

Netlist identical; ERC 333 -> 330 (the three lib_symbol_mismatch
warnings are gone); DRC with schematic parity unchanged.

Co-Authored-By: Claude Opus 5.5 <noreply@anthropic.com>
Parts:
- J7: symbol Connector:Micro_SD_Card_Det2 -> libreboard:Micro_SD_Card_Det2
Changed lines of the file:
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@@
 	)
 	(symbol
-		(lib_id "Connector:Micro_SD_Card_Det2")
+		(lib_id "libreboard:Micro_SD_Card_Det2")
 		(at 255.27 125.73 0)
 		(unit 1)

Commit message: BOM: J2 to a generic 2x7 header, J22 to the EDAC HDMI connector
JLC has no footprint for the Molex parts chosen before (C561778,
C5240402), so its preview could not show or place them.

- J2: BOOMELE 2.54-2*7P (C71397, gold, 21.5k at JLC). 6/3 mm pins and a
  2.5 mm insulator instead of the C-Grid's 6.1/2.8 mm and 2.29 mm.
- J22: EDAC 690-019-298-412 (C5291558, 1,850 at JLC), the part the
  footprint from Raspberry Pi's CM5 IO board was drawn for.

JLC's footprints for both match ours pad for pad. Neither part is at
DigiKey or Mouser, so Distributor = LCSC. Fields only: ERC (330) and DRC
with schematic parity (103, 4 parity) unchanged.

Co-Authored-By: Claude Opus 5.5 <noreply@anthropic.com>
Parts:
- J2: Dist. P/N 538-10-89-7142 -> C71397; Distributor Mouser -> LCSC; LCSC C561778 -> C71397; Manf. P/N 0010897142 -> 2.54-2*7PPin; Manufacturer Molex -> BOOMELE; Part Description Pin Header, Male, 2x07, 2.54mm P, Vertical, 15 uin gold -> Pin Header, Male, 2x07, 2.54mm P, Vertical, gold
Changed lines of the file:
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@@
 			)
 		)
-		(property "Datasheet" ""
+		(property "Datasheet" "https://www.lcsc.com/datasheet/lcsc_datasheet_2212121509_BOOMELE-Boom-Precision-Elec-2-54-2-7P_C71397.pdf"
 			(at 36.83 177.8 0)
 			(hide yes)
@@
 			)
 		)
-		(property "Part Description" "Pin Header, Male, 2x07, 2.54mm P, Vertical, 15 uin gold"
+		(property "Part Description" "Pin Header, Male, 2x07, 2.54mm P, Vertical, gold"
 			(at 36.83 177.8 0)
 			(hide yes)
@@
 			)
 		)
-		(property "Dist. P/N" "538-10-89-7142"
+		(property "Dist. P/N" "C71397"
 			(at 36.83 177.8 0)
 			(hide yes)
@@
 			)
 		)
-		(property "Distributor" "Mouser"
+		(property "Distributor" "LCSC"
 			(at 36.83 177.8 0)
 			(hide yes)
@@
 			)
 		)
-		(property "Manf. P/N" "0010897142"
+		(property "Manf. P/N" "2.54-2*7PPin"
 			(at 36.83 177.8 0)
 			(hide yes)
@@
 			)
 		)
-		(property "LCSC" "C561778"
+		(property "LCSC" "C71397"
 			(at 36.83 177.8 0)
 			(hide yes)
@@
 			)
 		)
-		(property "Manufacturer" "Molex"
+		(property "Manufacturer" "BOOMELE"
 			(at 36.83 177.8 0)
 			(hide yes)
