File: CM5_GPIO.kicad_sch (KiCad schematic)
At the start: 43 parts, among them J14 JST_BM04B-SRSS-TB, J16 JST_BM04B-SRSS-TB, J19 Conn_1x03_Male, J2 Conn_2x07_Male, J3 Conn_1x03_Male, J7 Micro_SD_Card_Det, J8 Conn_2x20_Male, SW1 Right angle Tact button, SW2 Right angle Tact button, U1 TPD4EUSB30, U16 SN74AHCT1G125DCKR, U17 TCA9538DBR, U18 RT9742GGJ5, U2 TPD4EUSB30, U3 LPJG0926HENL, U5 74LVC1G07SE-7, U9 SK6812

Commit message: BOM: C71 to a 10 V 10 uF 0402 (Murata GRM155R61A106ME11D)
C71 sits on +5v (5.19 V) and was a 6.3 V part shared with C34/C46.
Same footprint, so fields only: LCSC C408132, DigiKey
490-GRM155R61A106ME11DTR-ND. C34/C46 (1.2 V) keep the 6.3 V part.
ERC, DRC and schematic parity unchanged.

Co-Authored-By: Claude Opus 5.5 <noreply@anthropic.com>
Parts:
- C71: Dist. P/N 478-KGM05CR50J106MHTR-ND -> 490-GRM155R61A106ME11DTR-ND; LCSC C15525 -> C408132; Manf. P/N 04026D106MAT2A -> GRM155R61A106ME11D; Manufacturer Kyocera -> Murata; Part Description Capacitor, Ceramic, 10µF, ±20%, 6.3V, X5R, 0402 (1005m) -> Capacitor, Ceramic, 10µF, ±20%, 10V, X5R, 0402 (1005m)
Changed lines of the file:
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@@
 			)
 		)
-		(property "Part Description" "Capacitor, Ceramic, 10µF, ±20%, 6.3V, X5R, 0402 (1005m)"
+		(property "Part Description" "Capacitor, Ceramic, 10µF, ±20%, 10V, X5R, 0402 (1005m)"
 			(at 180.34 252.73 0)
 			(hide yes)
@@
 			)
 		)
-		(property "Dist. P/N" "478-KGM05CR50J106MHTR-ND"
+		(property "Dist. P/N" "490-GRM155R61A106ME11DTR-ND"
 			(at 180.34 252.73 0)
 			(hide yes)
@@
 			)
 		)
-		(property "Manf. P/N" "04026D106MAT2A"
+		(property "Manf. P/N" "GRM155R61A106ME11D"
 			(at 180.34 252.73 0)
 			(hide yes)
@@
 			)
 		)
-		(property "Manufacturer" "Kyocera"
+		(property "Manufacturer" "Murata"
 			(at 180.34 252.73 0)
 			(hide yes)
@@
 			)
 		)
-		(property "LCSC" "C15525"
+		(property "LCSC" "C408132"
 			(at 180.34 252.73 0)
 			(hide yes)
