File: PCIe-M2.kicad_sch (KiCad schematic)
At the start: 25 parts, among them J4 Bus_M.2_Socket_M, M1 M2x4mm screw, M2 M2-0.4mm nut, M3 M2-0.4mm nut, M4 M2-0.4mm nut, M5 M2-0.4mm nut, U7 ASEK-32.768KHZ-L-R-T, U8 AP3441SHE-7B

Commit message: BOM: LCSC codes for JLCPCB assembly, DigiKey numbers verified
Sourcing pass for a rev3 build at JLCPCB (SMT + through-hole), keeping
the DigiKey BOM usable. Report and per-part data in bom/rev3-sourcing.*.

- New hidden "LCSC" field on 189 parts (88 of 93 part numbers).
  Passives use JLC Basic/Preferred equivalents where value, size,
  tolerance, voltage and dielectric match or improve (0402 resistors at
  62.5 mW: worst-case dissipation on this board < 5 mW); ICs and
  connectors use the exact part. Exact codes are stored even where JLC
  has no stock (U4/U14, U3, U16, U17, BT1) - see the report.
- DigiKey: every existing number checked against its MPN (reel numbers
  kept). Filled: J7 (was Farnell 2358234), C60 (AVX new PN
  KGM05ACG1H6R8CH), C61, C66-C68, Q1/Q2, U20, U21. C73: wrong number
  (490-1494-2-ND is GRM188R71H102KA01D) cleared - to fill by hand.
- C72: Murata GRM188R71C104KA01D is obsolete -> Yageo CC0603KRX7R9BB104
  (0.1 uF 50 V X7R 0603).
- Fixes: L2/L3 manufacturer Coilcraft -> Bourns; U9 distributor typo
  LSCS -> LCSC; C27-C29 DigiKey number without " - Cut Tape" suffix.

Not yet stored: Y1, J2, J8, SW1/SW2 candidates need review; M1 is a
screw. Connectivity, values and footprints unchanged; ERC unchanged
at 342.

Co-Authored-By: Claude Opus 5.5 <noreply@anthropic.com>
Parts:
- C10, C19: LCSC (none) -> C1525
- C11: LCSC (none) -> C1538
- C14, C15, C16, C17, C4, C6: LCSC (none) -> C15850
- D3: LCSC (none) -> C125113
- J4: LCSC (none) -> C574849
- L1: LCSC (none) -> C22404330
- M2, M3, M4, M5: LCSC (none) -> C2916320
- R14: LCSC (none) -> C25741
- R15: LCSC (none) -> C25744
- R16: LCSC (none) -> C25879
- R17: LCSC (none) -> C11702
- U7: LCSC (none) -> C2650753
- U8: LCSC (none) -> C2070918
