File: libreboard.kicad_pcb (KiCad board)
At the start: 6 copper layers, 125 x 125 mm, 218 parts, among them J1 USB-C, J10 USB-C, J100 Screw Terminal, J101 Screw Terminal, J11 USB_C_Receptacle_USB2.0, J14 JST_BM04B-SRSS-TB, J15 USB_C_Receptacle, J16 JST_BM04B-SRSS-TB, J17 USB-C, J19 Conn_1x03_Male, J2 Conn_2x07_Male, J22 Conn_HDMI, J3 Conn_1x03_Male, J4 Bus_M.2_Socket_M, J5 Conn_1x22_Female, J51 12V Fan 1, J52 12V Fan 2, J53 12V Fan 3, J54 12V Fan 4, J6 USB-C, J7 Micro_SD_Card_Det, J8 Conn_2x20_Male, Q1 2N7002, Q2 2N7002, SW1 Right angle Tact button, SW2 Right angle Tact button, U1 TPD4EUSB30, U10 EMC2305-x-AP, U11 TUSB4041I, U12 RT9742SNGV, U13 TLV75712PDBVR, U14 TPS552892RYQR, U15 AP22653W6, U16 SN74AHCT1G125DRLR, U17 TCA9538DBR, U18 RT9742GGJ5, U19 TPS3808G01DBVR, U2 TPD4EUSB30, U20 LP38693MP-3.3, U21 HD3SS3220RNHR, U3 MagJack-A70-112-331N126, U4 TPS552892RYQR, U5 74LVC1G07SE-7, U6 AP22653W6, U7 ASEK-32.768KHZ-L-R-T, U8 AP3441SHE-7B, U9 SK6812, Y1 ECS-2520MV-240-CN-TR

Commit message: U3: MagJack TMJG4926HENL -> LINK-PP LPJG0926HENL (same pinout)
The Rev1 Ethernet fault was never a broken winding: the jacks fitted
(and the spares) are Taoglas TMJG0813GENL, which fits the same holes
but has a different pinout (4/5 = a signal pair, 9 = centre tap,
10 = GND, no pins 11-14). On our footprint that shorts one pair on
the CT net and puts TRD3 on the centre tap and ground, so 100 Mb/s
works and gigabit never can.

U3 now names LINK-PP LPJG0926HENL. Its datasheet (LP18022610 rev A)
has the same schematic, pin layout and footprint as TMJG4926HENL
(SPE-23-8-193-B): TD1-TD4 on 1/2, 3/6, 7/8, 9/10, CT 4/5, VC 11-14,
green LED 15/16, yellow 17/18. JLC C22457393, 2305 in stock; the
Taoglas part has 0 at JLC and 4 at DigiKey. Rated 0-70 C instead of
-40-85 C. Not found at DigiKey or Mouser, so Distributor = LCSC
(same convention as U9).

Fields changed on the symbol and the PCB footprint: Value,
Datasheet, Manufacturer, Manf. P/N, Distributor, Dist. P/N, LCSC,
and a Description note not to substitute TMJG0813GENL. Sourcing
report updated to match.

ERC 342 unchanged; DRC with schematic parity unchanged.

Co-Authored-By: Claude Opus 5.5 <noreply@anthropic.com>
Parts:
- U3: value MagJack-A70-112-331N126 -> LPJG0926HENL
Changed lines of the file:
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@@
 			)
 		)
-		(property "Value" "MagJack-A70-112-331N126"
+		(property "Value" "LPJG0926HENL"
 			(at 0 11.58 0)
 			(layer "F.Fab")
@@
 			)
 		)
-		(property "Datasheet" "https://www.taoglas.com/datasheets/TMJG4926HENL.pdf"
+		(property "Datasheet" "https://www.l-p.com/file/datasheet/lpjg0926henl.pdf"
 			(at 0 0 0)
 			(unlocked yes)
@@
 			)
 		)
-		(property "Description" ""
+		(property "Description" "RJ45 1G MagJack, LPJG0926HENL/TMJG4926HENL pinout (4,5 = CT; 9,10 = TD4; 11-14 = VC). Do not substitute TMJG0813GENL: different pinout (9 = CT, 10 = GND)."
 			(at 0 0 0)
 			(unlocked yes)
@@
 			)
 		)
-		(property "Dist. P/N" "931-TMJG4926HENL-ND"
+		(property "Dist. P/N" "C22457393"
 			(at 0 0 0)
 			(unlocked yes)
@@
 			)
 		)
-		(property "Distributor" "Digikey"
+		(property "Distributor" "LCSC"
 			(at 0 0 0)
 			(unlocked yes)
@@
 			)
 		)
-		(property "Manf. P/N" "TMJG4926HENL"
+		(property "Manf. P/N" "LPJG0926HENL"
 			(at 0 0 0)
 			(unlocked yes)
@@
 			)
 		)
-		(property "Manufacturer" "Taoglas Limited"
+		(property "Manufacturer" "LINK-PP"
 			(at 0 0 0)
 			(unlocked yes)
@@
 			)
 		)
-		(property "LCSC" "C37415176"
+		(property "LCSC" "C22457393"
 			(at 0 0 0)
 			(unlocked yes)
